Commit message: Unfinish: change to livox mid100

File: launch/include/config/robot.urdf.xacro (robot description, xacro)
@@ -19,5 +19,5 @@
     <parent link="chassis_link" />
     <child link="velodyne" />
-    <origin xyz="0 0 0" rpy="0 0 0" />
+    <origin xyz="1.1 1.4 1.35" rpy="0 0.53 0" />
   </joint>
   <link name="navsat_link"> </link>

Commit message: test IMU bag but rotation is still a problem

File: launch/include/config/robot.urdf.xacro (robot description, xacro)
@@ -13,5 +13,5 @@
     <parent link="chassis_link" />
     <child link="imu_link" />
-    <origin xyz="0 0 0" rpy="0 0 0" />
+    <origin xyz="-3.36 1.16 0" rpy="-3.142 0 0" />
   </joint>
   <link name="velodyne"> </link>
@@ -19,5 +19,5 @@
     <parent link="chassis_link" />
     <child link="velodyne" />
-    <origin xyz="1.1 1.4 1.35" rpy="0 0.53 0" />
+    <origin xyz="1.0 1.0 1.7" rpy="0 0.58 0" />
   </joint>
   <link name="navsat_link"> </link>

Commit message: before 5.1

File: launch/include/config/robot.urdf.xacro (robot description, xacro)
@@ -13,5 +13,5 @@
     <parent link="chassis_link" />
     <child link="imu_link" />
-    <origin xyz="-3.36 1.16 0" rpy="-3.142 0 0" />
+    <origin xyz="0 0 0" rpy="0 0 0" />
   </joint>
   <link name="velodyne"> </link>
@@ -19,5 +19,5 @@
     <parent link="chassis_link" />
     <child link="velodyne" />
-    <origin xyz="1.0 1.0 1.7" rpy="0 0.58 0" />
+    <origin xyz="0 0 0" rpy="0 0 0" />
   </joint>
   <link name="navsat_link"> </link>
